File: PCB/MoodBearsKB/MoodBearsKB.kicad_pcb (KiCad board)
At the start: 2 copper layers, 266.5 x 94.5 mm, 104 parts, among them J1 MJ-4PP-9, J2 MJ-4PP-9, U1 xiao-ble, U2 xiao-ble

Commit message: sent to PCBWay!
Parts:
- RSW1, RSW2: footprint Button_Switch_THT:SW_Tactile_SPST_Angled_PTS645Vx39-2LFS -> TOTEMlib:SKHLLCA010
- moved RSW1 2.48 mm to (123.0, 52.7)
- moved RSW2 2.46 mm to (177.0, 52.7)
- renumbered DL17 to DL16, DL16 to DL17, SWL17 to SWL16, SWL16 to SWL17
Connections:
- RSW1 pad 1: RESET_L -> GND_L
- RSW1 pad 2: GND_L -> RESET_L
- RSW2 pad 1: GND_R -> RESET_R
- RSW2 pad 2: RESET_R -> GND_R
Routing:
- net GND_L: vias 93 -> 94
