File: PCB/MoodBearsKB/MoodBearsKB.kicad_sch (KiCad schematic)
At the start: 92 parts, among them J1 MJ-4PP-9, J2 MJ-4PP-9, U1 xiao-ble, U2 xiao-ble

Commit message: sent to PCBWay!
Parts:
- RSW1, RSW2: footprint Button_Switch_THT:SW_Tactile_SPST_Angled_PTS645Vx39-2LFS -> TOTEMlib:SKHLLCA010
Connections:
- net GND_L: now also RSW1.1; no longer RSW1.2
- net GND_R: now also RSW2.2; no longer RSW2.1
- net RESET_L: now also RSW1.2; no longer RSW1.1
- net RESET_R: now also RSW2.1; no longer RSW2.2
Changed lines of the file:
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@@
 		(lib_id "Switch:SW_Push")
 		(at 127 67.31 0)
+		(mirror y)
 		(unit 1)
 		(exclude_from_sim no)
@@
 			)
 		)
-		(property "Footprint" "Button_Switch_THT:SW_Tactile_SPST_Angled_PTS645Vx39-2LFS"
+		(property "Footprint" "TOTEMlib:SKHLLCA010"
 			(at 127 62.23 0)
 			(effects
@@
 		(lib_id "Switch:SW_Push")
 		(at 171.45 67.31 0)
-		(mirror y)
 		(unit 1)
 		(exclude_from_sim no)
@@
 			)
 		)
-		(property "Footprint" "Button_Switch_THT:SW_Tactile_SPST_Angled_PTS645Vx39-2LFS"
+		(property "Footprint" "TOTEMlib:SKHLLCA010"
 			(at 171.45 62.23 0)
 			(effects

Commit message: Edit Schematic Footer
Other:
- note added: "MoodBearsKB"
- note removed: "T O T E M"
- company: (none) -> s-grundner
- title: TOTEM split keyboard -> Mood Bears Split Keyboard
Changed lines of the file:
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@@
 	(paper "A4")
 	(title_block
-		(title "TOTEM split keyboard")
+		(title "Mood Bears Split Keyboard")
 		(date "2025-06-10")
 		(rev "S.3")
-		(comment 1 "made by GEIST / edited by s-grundner")
+		(company "s-grundner")
+		(comment 1 "Based on the TOTEM by GEIST")
 	)
 	(rectangle
@@
 		)
 	)
-	(text "T O T E M"
-		(exclude_from_sim no)
-		(at 54.61 190.5 0)
-		(effects
-			(font
+	(text "MoodBearsKB"
+		(exclude_from_sim no)
+		(at 38.1 191.77 0)
+		(effects
+			(font
